File: Step 3: PCB Design/FelineWatchdog.kicad_pcb (KiCad board)
At the start: 2 copper layers, 38 x 65 mm, 29 parts, among them J1 USB_C_Receptacle_PowerOnly_6P, J12 Conn_01x04_Socket, J2 Conn_01x02_Socket, J3 Conn_01x02_Pin, Q2 FS8205A, SW1 RESET, U1 AMS1117-3.3, U3 TP4056, U4 DW01A, U5 ESP-32S

Commit message: Modified
Parts:
- added D1: SS14, Diode_SMD:D_SMA_Handsoldering, F.Cu at (154.3, 66.0)
- added D2: SS14, Diode_SMD:D_SMA_Handsoldering, F.Cu at (159.3, 74.0)
- added R2: 5k1, Resistor_SMD:R_0805_2012Metric_Pad1.20x1.40mm_HandSolder, F.Cu at (144.2, 80.5)
- added R3: 5k1, Resistor_SMD:R_0805_2012Metric_Pad1.20x1.40mm_HandSolder, F.Cu at (144.2, 77.7)
- U1: value AMS1117-3.3 -> AMS1117
Connections:
- J1 pad A5: unconnected-(J1-CC1-PadA5) -> Net-(J1-CC1)
- J1 pad B5: unconnected-(J1-CC2-PadB5) -> Net-(J1-CC2)
- R1 pad 1: +3.3V -> Net-(D1-K)
- U5 pad 2: +3.3V -> Net-(D1-K)
Routing:
- net Net-(D1-K): track 0.00 -> 51.1 mm
- net +3.3V: track 43.4 -> 20.3 mm
- net Net-(J1-CC2): track 0.00 -> 18.2 mm, vias 0 -> 2
- net Net-(J1-CC1): track 0.00 -> 16.5 mm, vias 0 -> 2
- net BATT +: track 36.2 -> 47.2 mm
- net +5V: track 104.6 -> 106.0 mm, vias 2 -> 4

Commit message: Modified
Parts:
- R9: value 1M -> 220
- U1: value AMS1117 -> AMS1117-3.3
Changed lines of the file:
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@@
 			)
 		)
-		(property "Value" "1M"
+		(property "Value" "220"
 			(at 0 1.65 0)
 			(layer "F.Fab")
@@
 			)
 		)
-		(property "Value" "AMS1117"
+		(property "Value" "AMS1117-3.3"
 			(at 5 -0.6 0)
 			(layer "F.SilkS")
