File: Step 3: PCB Design/FelineWatchdog.kicad_sch (KiCad schematic)
At the start: 29 parts, among them J1 USB_C_Receptacle_PowerOnly_6P, J12 Conn_01x04_Socket, J2 Conn_01x02_Socket, J3 Conn_01x02_Pin, J9 USB_B_Micro, Q2 FS8205A, SW1 RESET, U1 AMS1117-3.3, U2 ESP32-CAM, U3 TP4056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

Commit message: Modified
Parts:
- removed U2: ESP32-CAM, ESP32-CAM:ESP32-CAM, symbol ESP32-CAM:ESP32-CAM
- added D1, D2: SS14, Diode_SMD:D_SMA_Handsoldering, symbol Diode:SS14
- added R2, R3: 5k1, Resistor_SMD:R_0805_2012Metric_Pad1.20x1.40mm_HandSolder, symbol Device:R
Connections:
- net +3.3V: now also D1.2 (A); no longer R1.1, U5.2 (3V3)
- net BATT +: now also D2.2 (A)
- net GND: now also R2.2, R3.2
- net at J1.A5 (CC1): now also R2.1
- net at J1.B5 (CC2): now also R3.1
- new net: D1.1 (K), D2.1 (K), R1.1, U5.2 (3V3)
- no-connect marks 48 -> 38
Other:
- note removed: "ESP32-CAM"
- moved on the sheet: C2, C3, C4, D3, R1, R9, SW1, U1, U5

Commit message: Modified
Parts:
- R9: value 1M -> 220
Changed lines of the file:
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@@
 			)
 		)
-		(property "Value" "1M"
+		(property "Value" "220"
 			(at 139.446 167.64 0)
 			(effects
